File: thinkb/thinkb.kicad_pcb (KiCad board)
At the start: 2 copper layers, 293.5 x 138 mm, 127 parts, among them P1 battery+, P2 battery-, SW1 SW_Push, SW11 SW_Push, SW12 SW_Push, SW13 SW_Push, SW14 SW_Push, SW15 SW_Push, SW16 SW_Push, SW17 SW_Push, SW18 SW_Push, SW19 SW_Push, SW2 SW_Push, SW20 SW_Push, SW21 SW_Push, SW22 SW_Push, SW23 SW_Push, SW24 SW_Push, SW25 SW_Push, SW26 SW_Push, SW27 SW_Push, SW28 SW_Push, SW29 SW_Push, SW3 SW_Push, SW30 SW_Push, SW31 SW_Push, SW32 SW_Push, SW33 SW_Push, SW34 SW_Push, SW35 SW_Push, SW36 SW_Push, SW37 SW_Push, SW38 SW_Push, SW39 SW_Push, SW4 SW_Push, SW40 SW_Push, SW41 SW_Push, SW42 SW_Push, SW43 SW_Push, SW44 SW_Push, SW45 SW_Push, SW46 SW_Push, SW47 SW_Push, SW48 SW_Push, SW49 SW_Push, SW5 SW_Push, SW50 SW_Push, SW51 SW_Push, SW52 SW_Push, SW53 SW_Push, SW54 SW_Push, SW55 SW_Push, SW56 SW_Push, SW57 SW_Push, SW58 SW_Push, SW59 SW_Push, SW6 SW_Push, SW60 SW_Push, SW61 SW_Push, SW62 Reset, SW63 Power, SW7 SW_Push, SW8 SW_Push, SW9 SW_Push

Commit message: WIP
Parts:
- moved SW62 2.22 mm to (136.8, 39.9)
- moved SW63 1.62 mm to (170.8, 40.1)
Routing:
- net encA: track 0.00 -> 53.4 mm, vias 0 -> 1
- net encB: track 0.00 -> 43.5 mm, vias 0 -> 1
- net col0: track 412.6 -> 424.0 mm
- net col1: track 356.7 -> 366.1 mm
- net row4: track 451.1 -> 443.5 mm
- net col2: track 300.0 -> 307.3 mm
- net GND: track 0.00 -> 2.54 mm
- net row2: track 419.3 -> 421.3 mm
- net col4: track 220.7 -> 221.9 mm
Other:
- outline, holes or cut-outs redrawn

Commit message: Minor changes
Parts:
- moved P2 50.8 mm to (157.1, 99.9)
- moved P1 48.8 mm to (161.3, 99.9)
Connections:
- MCU1 pad 23: Net-(MCU1-Pad23) -> GND
- P2 pad 1: Net-(MCU1-Pad23) -> GND
Routing:
- net GND: track 2.54 -> 91.1 mm, vias 0 -> 1
- net Net-(P1-Pad1): track 0.00 -> 71.7 mm, vias 0 -> 2
- net Net-(MCU1-Pad22): track 0.00 -> 44.2 mm, vias 0 -> 1
- net Net-(MCU1-Pad24): track 0.00 -> 24.7 mm
Other:
- board text added: "+"
- board text added: "-"

Commit message: Corrected tracks by perimeter
Parts:
- moved SW2 12.1 mm to (80.8, 34.8)
- moved D32 12.1 mm to (115.7, 82.2)
- moved SW61 12.1 mm to (281.1, 84.6)
- moved SW6 12.1 mm to (286.7, 30.8)
- moved SW59 12.1 mm to (210.5, 98.9)
- moved SW29 12.1 mm to (273.1, 51.5)
- moved D39 12.1 mm to (98.8, 75.6)
- moved D19 12.1 mm to (229.3, 61.5)
- moved SW38 12.1 mm to (54.3, 68.0)
- moved D26 12.1 mm to (203.6, 109.8)
- moved D37 12.1 mm to (304.3, 65.6)
- moved SW3 12.1 mm to (115.8, 43.2)
- moved D12 12.1 mm to (242.2, 38.3)
- moved D15 12.1 mm to (84.7, 57.3)
- moved D3 12.1 mm to (123.6, 49.2)
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Routing:
- net col7: track 336.5 -> 326.2 mm
- net row4: track 443.5 -> 449.3 mm
- net col3: track 273.9 -> 268.2 mm
- net col0: track 424.0 -> 422.6 mm
- net col6: track 327.4 -> 326.4 mm

Commit message: New edge cuts
Parts:
- moved SW62 1.90 mm to (149.5, 39.9)
- moved SW63 1.75 mm to (182.7, 40.1)
Routing:
- net Net-(MCU1-Pad24): track 24.7 -> 26.4 mm
- net Net-(P1-Pad1): track 71.7 -> 73.5 mm
- net Net-(MCU1-Pad22): track 44.2 -> 45.6 mm
- net GND: track 91.1 -> 92.5 mm
Other:
- board size 293.5 x 138 mm -> 299.8 x 143 mm

Commit message: Mounting holes
Parts:
- added H1: MountingHole, MountingHole:MountingHole_2.2mm_M2, F.Cu at (165.7, 155.0)
- added H10: MountingHole, MountingHole:MountingHole_2.2mm_M2, F.Cu at (185.0, 78.4)
- added H11: MountingHole, MountingHole:MountingHole_2.2mm_M2, F.Cu at (292.4, 93.4)
- added H12: MountingHole, MountingHole:MountingHole_2.2mm_M2, F.Cu at (57.0, 19.3)
- added H13: MountingHole, MountingHole:MountingHole_2.2mm_M2, F.Cu at (96.9, 120.6)
- added H15: MountingHole, MountingHole:MountingHole_2.2mm_M2, F.Cu at (308.5, 70.8)
- added H16: MountingHole, MountingHole:MountingHole_2.2mm_M2, F.Cu at (30.9, 38.2)
- added H17: MountingHole, MountingHole:MountingHole_2.2mm_M2, F.Cu at (125.7, 139.9)
- added H18: MountingHole, MountingHole:MountingHole_2.2mm_M2, F.Cu at (203.7, 34.6)
- added H19: MountingHole, MountingHole:MountingHole_2.2mm_M2, F.Cu at (300.5, 37.7)
- added H2: MountingHole, MountingHole:MountingHole_2.2mm_M2, F.Cu at (205.9, 139.6)
- added H20: MountingHole, MountingHole:MountingHole_2.2mm_M2, F.Cu at (128.0, 34.5)
- added H21: MountingHole, MountingHole:MountingHole_2.2mm_M2, F.Cu at (239.5, 23.4)
- added H22: MountingHole, MountingHole:MountingHole_2.2mm_M2, F.Cu at (274.9, 19.4)
- added H3: MountingHole, MountingHole:MountingHole_2.2mm_M2, F.Cu at (38.9, 93.3)
- added H4: MountingHole, MountingHole:MountingHole_2.2mm_M2, F.Cu at (234.5, 120.4)
- added H5: MountingHole, MountingHole:MountingHole_2.2mm_M2, F.Cu at (23.1, 70.9)
- added H6: MountingHole, MountingHole:MountingHole_2.2mm_M2, F.Cu at (146.4, 78.4)
- added H7: MountingHole, MountingHole:MountingHole_2.2mm_M2, F.Cu at (264.8, 106.1)
- added H8: MountingHole, MountingHole:MountingHole_2.2mm_M2, F.Cu at (92.5, 23.2)
- added H9: MountingHole, MountingHole:MountingHole_2.2mm_M2, F.Cu at (67.1, 106.3)
Routing:
- net Net-(P1-Pad1): track 73.5 -> 76.4 mm
- net row1: track 374.2 -> 376.1 mm
- net row0: track 354.7 -> 356.6 mm
- net row2: track 421.3 -> 422.3 mm
Other:
- outline, holes or cut-outs redrawn

Commit message: Working on mounting holes
Parts:
- moved H16 0.50 mm to (30.9, 37.7)
- moved H9 0.36 mm to (66.8, 106.1)
- moved H17 0.30 mm to (125.7, 139.6)
- moved H8 0.20 mm to (92.5, 23.4)
- moved H4 0.20 mm to (234.5, 120.6)
- moved H7 0.10 mm to (264.7, 106.1)
- moved H11 0.10 mm to (292.4, 93.3)
- moved H5 0.10 mm to (23.1, 70.8)
- moved H20 0.10 mm to (128.0, 34.6)
- moved H12 0.10 mm to (57.0, 19.4)
Other:
- outline, holes or cut-outs redrawn

Commit message: Edges
Parts:
- moved D38 32.7 mm to (62.1, 41.3)
- moved D39 32.7 mm to (98.8, 42.9)
- moved D28 32.7 mm to (246.2, 22.2)
- moved D1 32.7 mm to (52.5, 4.08)
- moved SW58 32.7 mm to (240.3, 74.9)
- moved SW9 32.7 mm to (132.8, 16.7)
- moved SW12 32.7 mm to (232.5, 3.91)
- moved D53 32.7 mm to (308.3, 49.5)
- moved SW19 32.7 mm to (219.6, 27.1)
- moved D51 32.7 mm to (237.2, 61.9)
- moved SW54 32.7 mm to (50.3, 51.9)
- moved SW61 32.7 mm to (281.1, 51.9)
- moved D60 32.7 mm to (254.1, 55.3)
- moved H15 32.7 mm to (308.5, 38.1)
- moved SW51 32.7 mm to (227.5, 60.1)
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Other:
- board size 299.8 x 143 mm -> 298.9 x 143.1 mm

Commit message: Minor changes
Parts:
- moved ENC1 44.6 mm to (152.7, 111.3)
- moved SW43 44.6 mm to (210.8, 94.1)
- moved D45 44.6 mm to (291.1, 81.5)
- moved D28 44.6 mm to (250.5, 66.6)
- moved H9 44.6 mm to (71.1, 117.8)
- moved SW17 44.6 mm to (157.8, 141.7)
- moved SW19 44.6 mm to (223.9, 71.4)
- moved SW6 44.6 mm to (291.0, 42.5)
- moved D16 44.6 mm to (123.9, 77.4)
- moved D20 44.6 mm to (268.6, 64.8)
- moved SW11 44.6 mm to (202.9, 61.0)
- moved MCU1 44.6 mm to (170.0, 87.0)
- moved D38 44.6 mm to (66.4, 85.7)
- moved SW4 44.6 mm to (219.9, 54.9)
- moved D31 44.6 mm to (85.0, 85.5)
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Other:
- board size 298.9 x 143.1 mm -> 298.9 x 143 mm
