File: thinkb/thinkb.sch (KiCad schematic (older format))
At the start: 147 parts, among them P1 battery+, P2 battery-, SW1 SW_Push, SW11 SW_Push, SW12 SW_Push, SW13 SW_Push, SW14 SW_Push, SW15 SW_Push, SW16 SW_Push, SW17 SW_Push, SW18 SW_Push, SW19 SW_Push, SW2 SW_Push, SW20 SW_Push, SW21 SW_Push, SW22 SW_Push, SW23 SW_Push, SW24 SW_Push, SW25 SW_Push, SW26 SW_Push, SW27 SW_Push, SW28 SW_Push, SW29 SW_Push, SW3 SW_Push, SW30 SW_Push, SW31 SW_Push, SW32 SW_Push, SW33 SW_Push, SW34 SW_Push, SW35 SW_Push, SW36 SW_Push, SW37 SW_Push, SW38 SW_Push, SW39 SW_Push, SW4 SW_Push, SW40 SW_Push, SW41 SW_Push, SW42 SW_Push, SW43 SW_Push, SW44 SW_Push, SW45 SW_Push, SW46 SW_Push, SW47 SW_Push, SW48 SW_Push, SW49 SW_Push, SW5 SW_Push, SW50 SW_Push, SW51 SW_Push, SW52 SW_Push, SW53 SW_Push, SW54 SW_Push, SW55 SW_Push, SW56 SW_Push, SW57 SW_Push, SW58 SW_Push, SW59 SW_Push, SW6 SW_Push, SW60 SW_Push, SW61 SW_Push, SW62 Reset, SW63 Power, SW7 SW_Push, SW8 SW_Push, SW9 SW_Push

Commit message: Polishing
Parts:
- removed H17, H19, H23, H7, H8: MountingHole, MountingHole:MountingHole_2.2mm_M2, symbol Mechanical:MountingHole
- renumbered ENC2 to ENC1
Changed lines of the file:
@@
-$EndComp
-$Comp
-L Mechanical:MountingHole H8
-U 1 1 6154A57C
-P 7600 1350
-F 0 "H8" H 7700 1396 50  0000 L CNN
-F 1 "MountingHole" H 7700 1305 50  0000 L CNN
-F 2 "MountingHole:MountingHole_2.2mm_M2" H 7600 1350 50  0001 C CNN
-F 3 "~" H 7600 1350 50  0001 C CNN
-	1    7600 1350
-	1    0    0    -1
 $EndComp
 $Comp
@@
 F 3 "~" H 7600 1550 50  0001 C CNN
 	1    7600 1550
-	1    0    0    -1
-$EndComp
-$Comp
-L Mechanical:MountingHole H17
-U 1 1 6155803C
-P 7600 1950
-F 0 "H17" H 7700 1996 50  0000 L CNN
-F 1 "MountingHole" H 7700 1905 50  0000 L CNN
-F 2 "MountingHole:MountingHole_2.2mm_M2" H 7600 1950 50  0001 C CNN
-F 3 "~" H 7600 1950 50  0001 C CNN
-	1    7600 1950
 	1    0    0    -1
 $EndComp
@@
 $EndComp
 $Comp
-L Mechanical:MountingHole H7
-U 1 1 61591EB8
-P 9200 1150
-F 0 "H7" H 9300 1196 50  0000 L CNN
-F 1 "MountingHole" H 9300 1105 50  0000 L CNN
-F 2 "MountingHole:MountingHole_2.2mm_M2" H 9200 1150 50  0001 C CNN
-F 3 "~" H 9200 1150 50  0001 C CNN
-	1    9200 1150
-	1    0    0    -1
-$EndComp
-$Comp
 L Mechanical:MountingHole H10
 U 1 1 61591EBE
@@
 $EndComp
 $Comp
-L Mechanical:MountingHole H19
-U 1 1 61591ED0
-P 9200 1950
-F 0 "H19" H 9300 1996 50  0000 L CNN
-F 1 "MountingHole" H 9300 1905 50  0000 L CNN
-F 2 "MountingHole:MountingHole_2.2mm_M2" H 9200 1950 50  0001 C CNN
-F 3 "~" H 9200 1950 50  0001 C CNN
-	1    9200 1950
-	1    0    0    -1
-$EndComp
-$Comp
 L Mechanical:MountingHole H22
 U 1 1 61591ED6
@@
 $EndComp
 $Comp
-L evqwgd001:EVQWGD001 ENC2
+L evqwgd001:EVQWGD001 ENC1
 U 1 1 615A9AC4
 P 3550 850
-F 0 "ENC2" H 3828 904 50  0000 L CNN
+F 0 "ENC1" H 3828 904 50  0000 L CNN
 F 1 "EVQWGD001" H 3828 813 50  0000 L CNN
 F 2 "footprints:EVQWGD001" H 3550 850 50  0001 C CNN
@@
 Wire Wire Line
 	2900 750  3200 750
-$Comp
-L Mechanical:MountingHole H23
-U 1 1 61621F0C
-P 9200 2350
-F 0 "H23" H 9300 2396 50  0000 L CNN
-F 1 "MountingHole" H 9300 2305 50  0000 L CNN
-F 2 "MountingHole:MountingHole_2.2mm_M2" H 9200 2350 50  0001 C CNN
-F 3 "~" H 9200 2350 50  0001 C CNN
-	1    9200 2350
-	1    0    0    -1
-$EndComp
 $EndSCHEMATC
