File: top_cover/top_cover.kicad_pcb (KiCad board)
At the start: 2 copper layers, 341.3 x 148.9 mm, 77 parts, among them SW1 SW_Push, SW11 SW_Push, SW12 SW_Push, SW13 SW_Push, SW14 SW_Push, SW15 SW_Push, SW16 SW_Push, SW17 SW_Push, SW18 SW_Push, SW19 SW_Push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

Commit message: Renamed everything to chocofly
Other:
- board text added: "Chocofly"
