File: pcb/chocofly.kicad_pcb (KiCad board)
At the start: 2 copper layers, 242.8 x 295 mm, 148 parts, among them P1 battery+, P2 battery-, SW1 SW_Push, SW11 SW_Push, SW12 SW_Push, SW13 SW_Push, SW14 SW_Push, SW15 SW_Push, SW16 SW_Push, SW17 SW_Push, SW18 SW_Push, SW19 SW_Push, SW2 SW_Push, SW20 SW_Push, SW21 SW_Push, SW22 SW_Push, SW23 SW_Push, SW24 SW_Push, SW25 SW_Push, SW26 SW_Push, SW27 SW_Push, SW28 SW_Push, SW29 SW_Push, SW3 SW_Push, SW30 SW_Push, SW31 SW_Push, SW32 SW_Push, SW33 SW_Push, SW34 SW_Push, SW35 SW_Push, SW36 SW_Push, SW37 SW_Push, SW38 SW_Push, SW39 SW_Push, SW4 SW_Push, SW40 SW_Push, SW41 SW_Push, SW42 SW_Push, SW43 SW_Push, SW44 SW_Push, SW45 SW_Push, SW46 SW_Push, SW47 SW_Push, SW48 SW_Push, SW49 SW_Push, SW5 SW_Push, SW50 SW_Push, SW51 SW_Push, SW52 SW_Push, SW53 SW_Push, SW54 SW_Push, SW55 SW_Push, SW56 SW_Push, SW57 SW_Push, SW58 SW_Push, SW59 SW_Push, SW6 SW_Push, SW60 SW_Push, SW61 SW_Push, SW62 Reset, SW63 Power, SW7 SW_Push, SW8 SW_Push, SW9 SW_Push

Commit message: Routing the right half
Parts:
- moved D53 161.2 mm to (149.7, 32.5), turned to 270 degrees
- moved D6 158.8 mm to (149.7, -18.5), turned to 270 degrees
- moved D37 158.4 mm to (149.7, 15.5), turned to 270 degrees
- moved D21 157.6 mm to (149.7, -1.52), turned to 270 degrees
- moved H4 156.7 mm to (-139.5, 52.1), turned to 350.5 degrees
- moved H2 153.7 mm to (-138.5, 46.2), turned to 350.5 degrees
- moved H11 151.3 mm to (-133.7, 53.0), turned to 350.5 degrees
- moved SW46 151.0 mm to (-142.2, -19.4), turned to 341 degrees
- moved SW53 151.0 mm to (140.7, 28.0), turned to 0 degrees
- moved H1 150.9 mm to (-137.6, 40.3), turned to 350.5 degrees
- moved SW1 150.1 mm to (-125.5, -67.6), turned to 341 degrees
- moved SW6 150.1 mm to (140.7, -23.0), turned to 0 degrees
- moved SW30 148.5 mm to (-136.6, -35.4), turned to 341 degrees
- moved SW37 148.5 mm to (140.7, 11.0), turned to 0 degrees
- moved SW14 148.2 mm to (-131.1, -51.5), turned to 341 degrees
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Routing:
- net col7: track 43.9 -> 288.0 mm
- net row4: track 191.9 -> 294.0 mm
- net col3: track 207.8 -> 284.9 mm
- net row5: track 191.9 -> 266.3 mm
- net row6: track 173.0 -> 240.6 mm
- net row2: track 205.4 -> 272.2 mm
- net row1: track 226.4 -> 285.7 mm
- net row7: track 165.5 -> 218.0 mm
- net row0: track 222.4 -> 273.8 mm
- net row3: track 228.7 -> 267.0 mm
- net Net-(D17-Pad2): track 0.00 -> 26.6 mm
- net Net-(D53-Pad2): track 0.00 -> 26.6 mm
- net Net-(D6-Pad2): track 0.00 -> 26.6 mm
- net Net-(D61-Pad2): track 0.00 -> 26.6 mm
- net Net-(D37-Pad2): track 0.00 -> 26.6 mm
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Other:
- board size 242.8 x 295 mm -> 322.5 x 163.3 mm
- board text added: "Angle 9,5 degrees Angle 13,5 degrees"
- board text removed: "Angle 4 degrees Angle 13,5 degrees"

Commit message: WIP
Parts:
- moved D53 10.7 mm to (147.1, 42.8), turned to 266 degrees
- moved D6 10.5 mm to (150.6, -8.03), turned to 266 degrees
- moved D37 10.5 mm to (148.3, 25.9), turned to 266 degrees
- moved D21 10.5 mm to (149.5, 8.93), turned to 266 degrees
- moved H4 10.4 mm to (-142.8, 42.2), turned to 346.5 degrees
- moved H2 10.2 mm to (-141.4, 36.4), turned to 346.5 degrees
- moved H11 10.0 mm to (-137.0, 43.6), turned to 346.5 degrees
- moved SW46 10.0 mm to (-140.5, -29.2), turned to 337 degrees
- moved SW53 10.0 mm to (138.4, 37.7), turned to 356 degrees
- moved H1 10.0 mm to (-140.0, 30.6), turned to 346.5 degrees
- moved SW1 9.95 mm to (-120.5, -76.2), turned to 337 degrees
- moved SW6 9.95 mm to (142.0, -13.1), turned to 356 degrees
- moved SW30 9.85 mm to (-133.8, -44.9), turned to 337 degrees
- moved SW37 9.85 mm to (139.6, 20.8), turned to 356 degrees
- moved SW14 9.83 mm to (-127.2, -60.5), turned to 337 degrees
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Routing:
- net col5: track 47.8 -> 283.3 mm
- net col6: track 45.8 -> 274.3 mm
- net row0: track 273.8 -> 366.0 mm
- net row2: track 272.2 -> 364.0 mm
- net row1: track 285.7 -> 362.0 mm
- net row3: track 267.0 -> 294.2 mm
- net Net-(D35-Pad2): track 0.00 -> 26.6 mm
- net Net-(D28-Pad2): track 0.00 -> 26.6 mm
- net Net-(D27-Pad2): track 0.00 -> 26.6 mm
- net Net-(D20-Pad2): track 0.00 -> 26.6 mm
- net Net-(D11-Pad2): track 0.00 -> 26.6 mm
- net Net-(D59-Pad2): track 0.00 -> 26.6 mm
- net Net-(D51-Pad2): track 0.00 -> 26.6 mm
- net Net-(D4-Pad2): track 0.00 -> 26.6 mm
- net Net-(D5-Pad2): track 0.00 -> 26.6 mm
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Other:
- board size 322.5 x 163.3 mm -> 322.4 x 174.6 mm
