File: pcb/chocofly.kicad_pcb (KiCad board)
At the start: 2 copper layers, 322.4 x 174.6 mm, 148 parts, among them P1 battery+, P2 battery-, SW1 SW_Push, SW11 SW_Push, SW12 SW_Push, SW13 SW_Push, SW14 SW_Push, SW15 SW_Push, SW16 SW_Push, SW17 SW_Push, SW18 SW_Push, SW19 SW_Push, SW2 SW_Push, SW20 SW_Push, SW21 SW_Push, SW22 SW_Push, SW23 SW_Push, SW24 SW_Push, SW25 SW_Push, SW26 SW_Push, SW27 SW_Push, SW28 SW_Push, SW29 SW_Push, SW3 SW_Push, SW30 SW_Push, SW31 SW_Push, SW32 SW_Push, SW33 SW_Push, SW34 SW_Push, SW35 SW_Push, SW36 SW_Push, SW37 SW_Push, SW38 SW_Push, SW39 SW_Push, SW4 SW_Push, SW40 SW_Push, SW41 SW_Push, SW42 SW_Push, SW43 SW_Push, SW44 SW_Push, SW45 SW_Push, SW46 SW_Push, SW47 SW_Push, SW48 SW_Push, SW49 SW_Push, SW5 SW_Push, SW50 SW_Push, SW51 SW_Push, SW52 SW_Push, SW53 SW_Push, SW54 SW_Push, SW55 SW_Push, SW56 SW_Push, SW57 SW_Push, SW58 SW_Push, SW59 SW_Push, SW6 SW_Push, SW60 SW_Push, SW61 SW_Push, SW62 Reset, SW63 Power, SW7 SW_Push, SW8 SW_Push, SW9 SW_Push

Commit message: WIP
Routing:
- net row4: track 301.1 -> 389.9 mm
- net row7: track 225.1 -> 312.8 mm
- net row6: track 247.7 -> 335.2 mm
- net row5: track 280.0 -> 340.1 mm
- net row3: track 294.2 -> 352.8 mm
- net col4: track 49.8 -> 85.8 mm
- net Net-(D58-Pad2): track 0.00 -> 26.6 mm

Commit message: WIP
Parts:
- moved D53 36.0 mm to (133.0, 76.0), turned to 252.5 degrees
- moved D6 35.5 mm to (148.4, 27.4), turned to 252.5 degrees
- moved D37 35.4 mm to (138.1, 59.8), turned to 252.5 degrees
- moved D21 35.2 mm to (143.2, 43.6), turned to 252.5 degrees
- moved H4 35.0 mm to (-148.7, 7.69), turned to 333 degrees
- moved H2 34.3 mm to (-146.0, 2.39), turned to 333 degrees
- moved H11 33.8 mm to (-143.4, 10.4), turned to 333 degrees
- moved SW46 33.7 mm to (-129.8, -61.2), turned to 323.5 degrees
- moved SW53 33.7 mm to (125.8, 69.0), turned to 342.5 degrees
- moved H1 33.7 mm to (-143.3, -2.91), turned to 333 degrees
- moved SW1 33.5 mm to (-99.4, -102.2), turned to 323.5 degrees
- moved SW6 33.5 mm to (141.1, 20.4), turned to 342.5 degrees
- moved SW30 33.2 mm to (-119.6, -74.9), turned to 323.5 degrees
- moved SW37 33.2 mm to (130.9, 52.8), turned to 342.5 degrees
- moved SW14 33.1 mm to (-109.5, -88.5), turned to 323.5 degrees
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Routing:
- net col4: track 85.8 -> 117.8 mm
- net Net-(D50-Pad2): track 0.00 -> 26.6 mm
- net row6: track 335.2 -> 359.8 mm
Other:
- board size 322.4 x 174.6 mm -> 311.3 x 208.2 mm

Commit message: WIP
Parts:
- moved D53 71.5 mm to (84.0, 128.1), turned to 225.5 degrees
- moved D6 70.4 mm to (119.8, 91.7), turned to 225.5 degrees
- moved D37 70.3 mm to (95.9, 116.0), turned to 225.5 degrees
- moved D21 69.9 mm to (107.8, 103.8), turned to 225.5 degrees
- moved H4 69.5 mm to (-136.0, -60.7), turned to 306 degrees
- moved H2 68.2 mm to (-131.2, -64.2), turned to 306 degrees
- moved H11 67.1 mm to (-132.5, -55.9), turned to 306 degrees
- moved SW46 67.0 mm to (-87.8, -113.4), turned to 296.5 degrees
- moved SW53 67.0 mm to (80.8, 118.6), turned to 315.5 degrees
- moved H1 66.9 mm to (-126.4, -67.7), turned to 306 degrees
- moved SW1 66.6 mm to (-42.2, -136.2), turned to 296.5 degrees
- moved SW6 66.6 mm to (116.5, 82.2), turned to 315.5 degrees
- moved SW30 65.9 mm to (-72.6, -121.0), turned to 296.5 degrees
- moved SW37 65.9 mm to (92.7, 106.5), turned to 315.5 degrees
- moved SW14 65.8 mm to (-57.4, -128.6), turned to 296.5 degrees
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Routing:
- net col4: track 117.8 -> 278.7 mm
- net row4: track 389.9 -> 441.7 mm, vias 5 -> 6
- net row5: track 340.1 -> 385.4 mm
- net Net-(D26-Pad2): track 0.00 -> 26.6 mm
- net Net-(D18-Pad2): track 0.00 -> 26.6 mm
- net Net-(D42-Pad2): track 0.00 -> 26.6 mm
- net Net-(D34-Pad2): track 0.00 -> 26.6 mm
- net row2: track 364.0 -> 379.6 mm
- net Net-(ENC2-PadA): track 0.00 -> 12.4 mm
- net Net-(ENC2-PadB): track 0.00 -> 11.9 mm
- net Net-(D62-Pad2): track 0.00 -> 7.85 mm
- net row3: track 352.8 -> 356.3 mm
- net row1: track 362.0 -> 365.6 mm
Other:
- board size 311.3 x 208.2 mm -> 242.8 x 295 mm

Commit message: WIP
Parts:
- moved D53 139.1 mm to (153.0, 7.32), turned to 279.5 degrees
- moved D6 137.0 mm to (144.6, -43.0), turned to 279.5 degrees
- moved D37 136.7 mm to (150.2, -9.44), turned to 279.5 degrees
- moved D21 135.9 mm to (147.4, -26.2), turned to 279.5 degrees
- moved H4 135.2 mm to (-129.0, 74.4), turned to 0 degrees
- moved H2 132.6 mm to (-129.0, 68.4), turned to 0 degrees
- moved H11 130.6 mm to (-123.1, 74.4), turned to 0 degrees
- moved SW46 130.3 mm to (-143.4, 4.37), turned to 350.5 degrees
- moved SW53 130.3 mm to (143.4, 4.37), turned to 9.5 degrees
- moved H1 130.2 mm to (-129.0, 62.5), turned to 0 degrees
- moved SW1 129.5 mm to (-135.0, -45.9), turned to 350.5 degrees
- moved SW6 129.5 mm to (135.0, -45.9), turned to 9.5 degrees
- moved SW30 128.2 mm to (-140.6, -12.4), turned to 350.5 degrees
- moved SW37 128.2 mm to (140.6, -12.4), turned to 9.5 degrees
- moved SW14 127.9 mm to (-137.8, -29.2), turned to 350.5 degrees
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Routing:
- net row2: track 379.6 -> 484.8 mm, vias 6 -> 7
- net row3: track 356.3 -> 445.7 mm, vias 8 -> 9
- net row6: track 359.8 -> 435.7 mm
- net row7: track 312.8 -> 385.6 mm
- net encB: track 61.5 -> 127.9 mm, vias 1 -> 3
- net encA: track 65.4 -> 126.3 mm, vias 1 -> 3
- net col7: track 288.0 -> 348.6 mm
- net col0: track 293.8 -> 348.1 mm
- net col1: track 289.5 -> 343.0 mm
- net row5: track 385.4 -> 437.4 mm
- net col6: track 274.3 -> 326.0 mm
- net row4: track 441.7 -> 491.9 mm
- net col5: track 283.3 -> 324.1 mm
- net col2: track 297.4 -> 334.9 mm, vias 2 -> 3
- net row0: track 366.0 -> 392.6 mm, vias 3 -> 4
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Other:
- board size 242.8 x 295 mm -> 317 x 133.4 mm

Commit message: All connected
Parts:
- moved D53 36.0 mm to (147.1, 42.8), turned to 266 degrees
- moved D6 35.5 mm to (150.6, -8.03), turned to 266 degrees
- moved D37 35.4 mm to (148.3, 25.9), turned to 266 degrees
- moved D21 35.2 mm to (149.5, 8.93), turned to 266 degrees
- moved H4 35.0 mm to (-142.8, 42.2), turned to 346.5 degrees
- moved H2 34.3 mm to (-141.4, 36.4), turned to 346.5 degrees
- moved H11 33.8 mm to (-137.0, 43.6), turned to 346.5 degrees
- moved SW46 33.7 mm to (-140.5, -29.2), turned to 337 degrees
- moved SW53 33.7 mm to (138.4, 37.7), turned to 356 degrees
- moved H1 33.7 mm to (-140.0, 30.6), turned to 346.5 degrees
- moved SW1 33.5 mm to (-120.5, -76.2), turned to 337 degrees
- moved SW6 33.5 mm to (142.0, -13.1), turned to 356 degrees
- moved SW30 33.2 mm to (-133.8, -44.9), turned to 337 degrees
- moved SW37 33.2 mm to (139.6, 20.8), turned to 356 degrees
- moved SW14 33.1 mm to (-127.2, -60.5), turned to 337 degrees
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Routing:
- net col0: track 348.1 -> 463.5 mm
- net col1: track 343.0 -> 417.7 mm, vias 2 -> 3
- net col7: track 348.6 -> 406.6 mm
- net row1: track 387.3 -> 445.0 mm, vias 5 -> 7
- net GND: track 80.8 -> 136.5 mm, vias 2 -> 4
- net col6: track 326.0 -> 368.0 mm, vias 2 -> 3
- net col2: track 334.9 -> 369.9 mm
- net row0: track 392.6 -> 413.2 mm, vias 4 -> 5
- net Net-(P1-Pad1): track 6.10 -> 21.9 mm, vias 0 -> 1
- net Net-(MCU1-Pad24): track 24.0 -> 38.2 mm
- net Net-(MCU1-Pad22): track 14.9 -> 17.1 mm
Other:
- board size 317 x 133.4 mm -> 322.4 x 174.6 mm

Commit message: All cleaned up
Parts:
- moved D53 36.0 mm to (153.0, 7.32), turned to 279.5 degrees
- moved D6 35.5 mm to (144.6, -43.0), turned to 279.5 degrees
- moved D37 35.4 mm to (150.2, -9.44), turned to 279.5 degrees
- moved D21 35.2 mm to (147.4, -26.2), turned to 279.5 degrees
- moved H4 35.0 mm to (-129.0, 74.4), turned to 0 degrees
- moved H2 34.3 mm to (-129.0, 68.4), turned to 0 degrees
- moved H11 33.8 mm to (-123.1, 74.4), turned to 0 degrees
- moved SW46 33.7 mm to (-143.4, 4.37), turned to 350.5 degrees
- moved SW53 33.7 mm to (143.4, 4.37), turned to 9.5 degrees
- moved H1 33.7 mm to (-129.0, 62.5), turned to 0 degrees
- moved SW1 33.5 mm to (-135.0, -45.9), turned to 350.5 degrees
- moved SW6 33.5 mm to (135.0, -45.9), turned to 9.5 degrees
- moved SW30 33.2 mm to (-140.6, -12.4), turned to 350.5 degrees
- moved SW37 33.2 mm to (140.6, -12.4), turned to 9.5 degrees
- moved SW14 33.1 mm to (-137.8, -29.2), turned to 350.5 degrees
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Routing:
- net encB: track 127.9 -> 123.3 mm
- net Net-(MCU1-Pad22): track 17.1 -> 16.3 mm
- net row3: vias 9 -> 8
- net row2: vias 7 -> 6
Other:
- board size 322.4 x 174.6 mm -> 317 x 133.4 mm

Commit message: WIP
Parts:
- moved D53 36.0 mm to (147.1, 42.8), turned to 266 degrees
- moved D6 35.5 mm to (150.6, -8.03), turned to 266 degrees
- moved D37 35.4 mm to (148.3, 25.9), turned to 266 degrees
- moved D21 35.2 mm to (149.5, 8.93), turned to 266 degrees
- moved H4 35.0 mm to (-142.8, 42.2), turned to 346.5 degrees
- moved H2 34.3 mm to (-141.4, 36.4), turned to 346.5 degrees
- moved H11 33.8 mm to (-137.0, 43.6), turned to 346.5 degrees
- moved SW46 33.7 mm to (-140.5, -29.2), turned to 337 degrees
- moved SW53 33.7 mm to (138.4, 37.7), turned to 356 degrees
- moved H1 33.7 mm to (-140.0, 30.6), turned to 346.5 degrees
- moved SW1 33.5 mm to (-120.5, -76.2), turned to 337 degrees
- moved SW6 33.5 mm to (142.0, -13.1), turned to 356 degrees
- moved SW30 33.2 mm to (-133.8, -44.9), turned to 337 degrees
- moved SW37 33.2 mm to (139.6, 20.8), turned to 356 degrees
- moved SW14 33.1 mm to (-127.2, -60.5), turned to 337 degrees
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Routing:
- net Net-(D3-Pad2): track 26.6 -> 35.2 mm
- net Net-(D9-Pad2): track 26.6 -> 35.1 mm
- net Net-(D11-Pad2): track 26.6 -> 34.8 mm
- net Net-(D7-Pad2): track 26.6 -> 34.7 mm
- net Net-(D4-Pad2): track 26.6 -> 34.5 mm, vias 0 -> 1
- net col1: track 417.7 -> 423.8 mm
- net col0: track 463.5 -> 469.4 mm
- net col6: track 368.0 -> 372.5 mm
- net row1: track 444.8 -> 441.8 mm
- net col2: track 369.9 -> 371.1 mm
- net row0: track 413.2 -> 412.5 mm
Other:
- board size 317 x 133.4 mm -> 322.4 x 174.6 mm

Commit message: New break-off way
Parts:
- added H14: 1mm, footprints:hole_1mm, F.Cu at (-65.3, -61.9)
- added H17: 15mm, footprints:hole_15mm, F.Cu at (-25.3, -22.6)
- added H19: 15mm, footprints:hole_15mm, F.Cu at (0.71, -61.9)
- added H23: 15mm, footprints:hole_15mm, F.Cu at (16.7, -59.9)
- added H24: 10mm, footprints:hole_10mm, F.Cu at (-1.79, -49.9)
- added H25: 10mm, footprints:hole_10mm, F.Cu at (-1.79, -47.9)
- added H26: 10mm, footprints:hole_10mm, F.Cu at (-1.79, -53.9)
- added H27: 10mm, footprints:hole_10mm, F.Cu at (-1.79, -51.9)
- added H28: 10mm, footprints:hole_10mm, F.Cu at (-1.79, -45.9)
- added H29: 10mm, footprints:hole_10mm, F.Cu at (9.21, -53.9)
- added H30: 5mm, footprints:hole_5mm, F.Cu at (11.7, -55.9)
- added H31: 5mm, footprints:hole_5mm, F.Cu at (17.7, -55.9)
- added H32: 5mm, footprints:hole_5mm, F.Cu at (17.7, -53.9)
- added H33: 5mm, footprints:hole_5mm, F.Cu at (6.71, -51.9)
- added H34: 5mm, footprints:hole_5mm, F.Cu at (17.7, -57.9)
- added H35: 5mm, footprints:hole_5mm, F.Cu at (12.7, -51.9)
- added H36: 3mm, footprints:hole_3mm, F.Cu at (5.71, -49.9)
- added H37: 3mm, footprints:hole_3mm, F.Cu at (9.71, -49.9)
- added H38: 3mm, footprints:hole_3mm, F.Cu at (13.7, -49.9)
- added H39: 3mm, footprints:hole_3mm, F.Cu at (5.71, -47.9)
- added H40: 3mm, footprints:hole_3mm, F.Cu at (9.71, -47.9)
- added H41: 3mm, footprints:hole_3mm, F.Cu at (5.71, -45.9)
- added H42: 2mm, footprints:hole_2mm, F.Cu at (13.2, -57.9)
- added H43: 2mm, footprints:hole_2mm, F.Cu at (9.21, -45.9)
- added H44: 2mm, footprints:hole_2mm, F.Cu at (10.2, -57.9)
- added H45: 2mm, footprints:hole_2mm, F.Cu at (13.2, -47.9)
- added H46: 2mm, footprints:hole_2mm, F.Cu at (17.2, -51.9)
- added H47: 2mm, footprints:hole_2mm, F.Cu at (22.2, -57.9)
- added H48: 1mm, footprints:hole_1mm, F.Cu at (21.7, -53.9)
- added H49: 1mm, footprints:hole_1mm, F.Cu at (16.7, -49.9)
- added H5: 5mm, footprints:hole_5mm, F.Cu at (-82.0, -36.2)
- added H50: 1mm, footprints:hole_1mm, F.Cu at (11.7, -45.9)
- added H51: 1mm, footprints:hole_1mm, F.Cu at (21.7, -55.9)
- added H7: 3mm, footprints:hole_3mm, F.Cu at (-73.3, -59.9)
- added H8: 3mm, footprints:hole_3mm, F.Cu at (-75.2, -34.6)
- added H9: 3mm, footprints:hole_3mm, F.Cu at (-40.4, -26.2)
- H1, H2, H3: value MountingHole -> 10mm; footprint MountingHole:MountingHole_2.2mm_M2 -> footprints:hole_10mm
- H10, H11, H12: value MountingHole -> 2mm; footprint MountingHole:MountingHole_2.2mm_M2 -> footprints:hole_2mm
- H13: value MountingHole -> 1mm; footprint MountingHole:MountingHole_2.2mm_M2 -> footprints:hole_1mm
- H15, H16, H18, H20, H21, H22: value MountingHole -> 15mm; footprint MountingHole:MountingHole_2.2mm_M2 -> footprints:hole_15mm
- H4, H6: value MountingHole -> 5mm; footprint MountingHole:MountingHole_2.2mm_M2 -> footprints:hole_5mm
- moved H21 170.3 mm to (16.7, -61.9), turned to 0 degrees
- moved H20 165.0 mm to (0.71, -59.9), turned to 0 degrees
- moved H22 160.2 mm to (0.71, -57.9), turned to 0 degrees
- moved H18 149.4 mm to (0.71, -55.9), turned to 0 degrees
- moved H2 137.9 mm to (-15.8, -20.3)
- moved H15 132.1 mm to (-50.3, -59.4), turned to 0 degrees
- moved H16 122.6 mm to (-50.3, -57.4), turned to 0 degrees
- moved H11 120.1 mm to (-72.8, -57.9), turned to 0 degrees
- moved H6 116.2 mm to (-38.3, -25.7)
- moved H1 111.0 mm to (-45.4, -27.4)
- moved H10 105.4 mm to (-75.8, -57.9), turned to 0 degrees
- moved H4 103.5 mm to (-72.8, -34.0)
- moved H3 98.4 mm to (-58.3, -30.5)
- moved H12 97.4 mm to (-63.0, -31.7)
- moved H13 87.3 mm to (-67.4, -32.7)
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Routing:
- net Net-(D13-Pad2): track 26.6 -> 34.6 mm
- net Net-(D5-Pad2): track 26.6 -> 33.0 mm
- net col7: track 406.6 -> 408.4 mm
- net row1: track 441.8 -> 443.1 mm
- net col6: track 372.5 -> 373.6 mm
Other:
- board size 322.4 x 174.6 mm -> 317 x 133.4 mm
