File: pcb_mx/chocofly.kicad_pcb (KiCad board)
At the start: 2 copper layers, 304 x 133.5 mm, 134 parts, among them P1 battery+, P2 battery-, SW1 SW_Push, SW11 SW_Push, SW12 SW_Push, SW13 SW_Push, SW14 SW_Push, SW15 SW_Push, SW16 SW_Push, SW17 SW_Push, SW18 SW_Push, SW19 SW_Push, SW2 SW_Push, SW20 SW_Push, SW21 SW_Push, SW22 SW_Push, SW23 SW_Push, SW24 SW_Push, SW25 SW_Push, SW26 SW_Push, SW27 SW_Push, SW28 SW_Push, SW29 SW_Push, SW3 SW_Push, SW30 SW_Push, SW31 SW_Push, SW32 SW_Push, SW33 SW_Push, SW34 SW_Push, SW35 SW_Push, SW36 SW_Push, SW37 SW_Push, SW38 SW_Push, SW39 SW_Push, SW4 SW_Push, SW40 SW_Push, SW41 SW_Push, SW42 SW_Push, SW43 SW_Push, SW44 SW_Push, SW45 SW_Push, SW46 SW_Push, SW47 SW_Push, SW48 SW_Push, SW49 SW_Push, SW5 SW_Push, SW50 SW_Push, SW51 SW_Push, SW52 SW_Push, SW53 SW_Push, SW54 SW_Push, SW55 SW_Push, SW56 SW_Push, SW57 SW_Push, SW58 SW_Push, SW59 SW_Push, SW6 SW_Push, SW60 SW_Push, SW61 SW_Push, SW62 Reset, SW63 Power, SW64 Power, SW7 SW_Push, SW8 SW_Push, SW9 SW_Push

Commit message: WIP on mx version of chocofly
Parts:
- added SW32: SW_Push, footprints:CherryMX_MidHeight_Hotswap_1u, F.Cu at (-103.6, 412.4)
- added SW32: SW_Push, footprints:CherryMX_MidHeight_Hotswap_1u, F.Cu at (-132.5, 449.8)
- added SW32: SW_Push, footprints:CherryMX_MidHeight_Hotswap_1u, F.Cu at (-57.4, 464.7)
- added SW32: SW_Push, footprints:CherryMX_MidHeight_Hotswap_1u, F.Cu at (-52.6, 493.6)
- added SW32: SW_Push, footprints:CherryMX_MidHeight_Hotswap_1u, F.Cu at (-145.0, 409.1)
- added SW32: SW_Push, footprints:CherryMX_MidHeight_Hotswap_1u, F.Cu at (-99.1, 393.9)
- added SW32: SW_Push, footprints:CherryMX_MidHeight_Hotswap_1u, F.Cu at (-62.1, 402.8)
- added SW32: SW_Push, footprints:CherryMX_MidHeight_Hotswap_1u, F.Cu at (-151.3, 446.6)
- added SW32: SW_Push, footprints:CherryMX_MidHeight_Hotswap_1u, F.Cu at (-129.4, 431.0)
- added SW32: SW_Push, footprints:CherryMX_MidHeight_Hotswap_1u, F.Cu at (-22.8, 497.9)
- added SW32: SW_Push, footprints:CherryMX_MidHeight_Hotswap_1u, F.Cu at (-48.5, 427.7)
- added SW32: SW_Push, footprints:CherryMX_MidHeight_Hotswap_1u, F.Cu at (-80.0, 395.9)
- added SW32: SW_Push, footprints:CherryMX_MidHeight_Hotswap_1u, F.Cu at (-90.0, 474.5)
- added SW32: SW_Push, footprints:CherryMX_MidHeight_Hotswap_1u, F.Cu at (-93.4, 451.5)
- added SW32: SW_Push, footprints:CherryMX_MidHeight_Hotswap_1u, F.Cu at (-84.5, 414.4)
- added SW32: SW_Push, footprints:CherryMX_MidHeight_Hotswap_1u, F.Cu at (-66.5, 421.3)
- added SW32: SW_Push, footprints:CherryMX_MidHeight_Hotswap_1u, F.Cu at (-38.2, 509.1)
- added SW32: SW_Push, footprints:CherryMX_MidHeight_Hotswap_1u, F.Cu at (-88.9, 433.0)
- added SW32: SW_Push, footprints:CherryMX_MidHeight_Hotswap_1u, F.Cu at (-112.5, 449.5)
- added SW32: SW_Push, footprints:CherryMX_MidHeight_Hotswap_1u, F.Cu at (-70.2, 481.8)
- added SW32: SW_Push, footprints:CherryMX_MidHeight_Hotswap_1u, F.Cu at (-108.0, 430.9)
- added SW32: SW_Push, footprints:CherryMX_MidHeight_Hotswap_1u, F.Cu at (-126.2, 412.2)
- added SW32: SW_Push, footprints:CherryMX_MidHeight_Hotswap_1u, F.Cu at (-52.9, 446.2)
- added SW32: SW_Push, footprints:CherryMX_MidHeight_Hotswap_1u, F.Cu at (-123.1, 393.4)
- added SW32: SW_Push, footprints:CherryMX_MidHeight_Hotswap_1u, B.Cu at (44.0, 409.2)
- added SW32: SW_Push, footprints:CherryMX_MidHeight_Hotswap_1u, B.Cu at (132.5, 449.8)
- added SW32: SW_Push, footprints:CherryMX_MidHeight_Hotswap_1u, B.Cu at (148.1, 427.8)
- added SW32: SW_Push, footprints:CherryMX_MidHeight_Hotswap_1u, B.Cu at (145.0, 409.1)
- added SW32: SW_Push, footprints:CherryMX_MidHeight_Hotswap_1u, B.Cu at (151.3, 446.6)
- added SW32: SW_Push, footprints:CherryMX_MidHeight_Hotswap_1u, B.Cu at (40.2, 479.1)
- added SW32: SW_Push, footprints:CherryMX_MidHeight_Hotswap_1u, B.Cu at (84.5, 414.4)
- added SW32: SW_Push, footprints:CherryMX_MidHeight_Hotswap_1u, B.Cu at (38.2, 509.1)
- added SW32: SW_Push, footprints:CherryMX_MidHeight_Hotswap_1u, F.Cu at (-71.0, 439.8)
- added SW32: SW_Push, footprints:CherryMX_MidHeight_Hotswap_1u, B.Cu at (52.6, 493.6)
- added SW32: SW_Push, footprints:CherryMX_MidHeight_Hotswap_1u, B.Cu at (62.1, 402.8)
- added SW32: SW_Push, footprints:CherryMX_MidHeight_Hotswap_1u, B.Cu at (99.1, 393.9)
- added SW32: SW_Push, footprints:CherryMX_MidHeight_Hotswap_1u, B.Cu at (141.9, 390.3)
- added SW32: SW_Push, footprints:CherryMX_MidHeight_Hotswap_1u, B.Cu at (93.4, 451.5)
- added SW32: SW_Push, footprints:CherryMX_MidHeight_Hotswap_1u, B.Cu at (90.0, 474.5)
- added SW32: SW_Push, footprints:CherryMX_MidHeight_Hotswap_1u, B.Cu at (108.0, 430.9)
- added SW32: SW_Push, footprints:CherryMX_MidHeight_Hotswap_1u, B.Cu at (88.9, 433.0)
- added SW32: SW_Push, footprints:CherryMX_MidHeight_Hotswap_1u, B.Cu at (129.4, 431.0)
- added SW32: SW_Push, footprints:CherryMX_MidHeight_Hotswap_1u, B.Cu at (71.0, 439.8)
- added SW32: SW_Push, footprints:CherryMX_MidHeight_Hotswap_1u, F.Cu at (-75.4, 458.4)
- added SW32: SW_Push, footprints:CherryMX_MidHeight_Hotswap_1u, B.Cu at (22.8, 497.9)
- added SW32: SW_Push, footprints:CherryMX_MidHeight_Hotswap_1u, B.Cu at (123.1, 393.4)
- added SW32: SW_Push, footprints:CherryMX_MidHeight_Hotswap_1u, B.Cu at (112.5, 449.5)
- added SW32: SW_Push, footprints:CherryMX_MidHeight_Hotswap_1u, B.Cu at (126.2, 412.2)
- added SW32: SW_Push, footprints:CherryMX_MidHeight_Hotswap_1u, B.Cu at (66.5, 421.3)
- added SW32: SW_Push, footprints:CherryMX_MidHeight_Hotswap_1u, B.Cu at (52.9, 446.2)
- added SW32: SW_Push, footprints:CherryMX_MidHeight_Hotswap_1u, B.Cu at (75.4, 458.4)
- added SW32: SW_Push, footprints:CherryMX_MidHeight_Hotswap_1u, B.Cu at (80.0, 395.9)
- added SW32: SW_Push, footprints:CherryMX_MidHeight_Hotswap_1u, B.Cu at (70.2, 481.8)
- added SW32: SW_Push, footprints:CherryMX_MidHeight_Hotswap_1u, B.Cu at (57.4, 464.7)
- added SW32: SW_Push, footprints:CherryMX_MidHeight_Hotswap_1u, F.Cu at (-40.2, 479.1)
- added SW32: SW_Push, footprints:CherryMX_MidHeight_Hotswap_1u, B.Cu at (48.5, 427.7)
- added SW32: SW_Push, footprints:CherryMX_MidHeight_Hotswap_1u, B.Cu at (103.6, 412.4)
- added SW32: SW_Push, footprints:CherryMX_MidHeight_Hotswap_1u, F.Cu at (-148.1, 427.8)
- added SW32: SW_Push, footprints:CherryMX_MidHeight_Hotswap_1u, F.Cu at (-141.9, 390.3)
- added SW32: SW_Push, footprints:CherryMX_MidHeight_Hotswap_1u, F.Cu at (-44.0, 409.2)
Other:
- board size 304 x 133.5 mm -> 330.4 x 635.7 mm
