File: pcb_mx/chocofly.kicad_pcb (KiCad board)
At the start: 2 copper layers, 330.4 x 635.7 mm, 194 parts, among them P1 battery+, P2 battery-, SW1 SW_Push, SW11 SW_Push, SW12 SW_Push, SW13 SW_Push, SW14 SW_Push, SW15 SW_Push, SW16 SW_Push, SW17 SW_Push, SW18 SW_Push, SW19 SW_Push, SW2 SW_Push, SW20 SW_Push, SW21 SW_Push, SW22 SW_Push, SW23 SW_Push, SW24 SW_Push, SW25 SW_Push, SW26 SW_Push, SW27 SW_Push, SW28 SW_Push, SW29 SW_Push, SW3 SW_Push, SW30 SW_Push, SW31 SW_Push, SW32 SW_Push, SW33 SW_Push, SW34 SW_Push, SW35 SW_Push, SW36 SW_Push, SW37 SW_Push, SW38 SW_Push, SW39 SW_Push, SW4 SW_Push, SW40 SW_Push, SW41 SW_Push, SW42 SW_Push, SW43 SW_Push, SW44 SW_Push, SW45 SW_Push, SW46 SW_Push, SW47 SW_Push, SW48 SW_Push, SW49 SW_Push, SW5 SW_Push, SW50 SW_Push, SW51 SW_Push, SW52 SW_Push, SW53 SW_Push, SW54 SW_Push, SW55 SW_Push, SW56 SW_Push, SW57 SW_Push, SW58 SW_Push, SW59 SW_Push, SW6 SW_Push, SW60 SW_Push, SW61 SW_Push, SW62 Reset, SW63 Power, SW64 Power, SW7 SW_Push, SW8 SW_Push, SW9 SW_Push

Commit message: wip
Parts:
- ENC1, ENC2: value EVQWGD001 -> EVQWGD001_for_mx; footprint footprints:EVQWGD001 -> footprints:EVQWGD001_for_mx
- moved ENC2 496.9 mm to (27.9, 464.6)
- moved ENC1 496.9 mm to (-27.9, 464.6)
- moved D33 495.9 mm to (-30.7, 515.4)
- moved D17 493.9 mm to (-15.3, 504.2)
- moved D34 493.6 mm to (41.9, 500.0)
- moved D18 492.7 mm to (26.5, 488.8)
- moved D62 492.3 mm to (33.5, 456.6)
- moved JP4 492.3 mm to (25.8, 447.6)
- moved JP3 492.3 mm to (27.1, 449.1)
- moved D41 491.5 mm to (-43.8, 497.9)
- moved D10 491.4 mm to (-19.0, 468.9)
- moved JP1 491.4 mm to (-11.4, 459.9)
- moved JP2 491.4 mm to (-12.7, 461.4)
- moved D42 490.5 mm to (58.3, 485.5)
- moved D25 490.3 mm to (-31.4, 483.4)
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Routing:
- net Net-(ENC2-PadA): track 11.7 -> 0.00 mm
- net Net-(ENC2-PadB): track 10.9 -> 0.00 mm
- net encA: track 124.0 -> 117.2 mm, vias 3 -> 2
- net row1: track 387.9 -> 382.7 mm
- net GND: track 134.0 -> 129.6 mm
- net encB: track 108.4 -> 104.0 mm, vias 3 -> 2
- net Net-(D62-A): track 3.62 -> 0.00 mm
- net row5: track 407.3 -> 405.2 mm

Commit message: wip
Parts:
- removed SW1, SW11, SW12, SW13, SW14, SW15, SW16, SW17, SW18, SW19, SW2, SW20, SW21, SW22, SW23, SW24, SW25, SW26, SW27, SW28, SW29, SW3, SW30, SW31, SW33, SW34, SW35, SW36, SW37, SW38, SW39, SW4, SW40, SW41, SW42, SW43, SW44, SW45, SW46, SW47, SW48, SW49, SW5, SW50, SW51, SW52, SW53, SW54, SW55, SW56, SW57, SW58, SW59, SW6, SW60, SW61, SW7, SW8, SW9: SW_Push, footprints:Kailh_socket_PG1350_chosfox_17_5mm
- removed the SW32 at (-65.2, -55.4)
- moved MCU1 494.0 mm to (-0.00, 439.5)
- moved P1 494.0 mm to (4.00, 422.9)
- moved P2 494.0 mm to (-4.00, 422.9)
- moved SW62 493.8 mm to (-23.9, 420.1)
- moved SW64 493.1 mm to (14.8, 411.1)
- moved SW63 474.0 mm to (23.4, 400.4)
- moved JP3 15.8 mm to (37.9, 460.7)
- moved JP4 15.8 mm to (36.6, 459.1)
- moved JP1 15.7 mm to (-21.0, 472.2)
- moved JP2 15.7 mm to (-22.4, 473.8)
Routing:
- net col7: track 488.4 -> 27.7 mm, vias 2 -> 1
- net col0: track 432.9 -> 22.7 mm
- net col2: track 411.8 -> 34.7 mm, vias 3 -> 1
- net col6: track 396.6 -> 28.6 mm, vias 3 -> 1
- net row4: track 466.1 -> 102.0 mm, vias 6 -> 5
- net row6: track 395.1 -> 77.7 mm
- net row5: track 405.2 -> 91.8 mm, vias 6 -> 5
- net col1: track 337.1 -> 25.0 mm
- net row2: track 463.8 -> 153.3 mm, vias 6 -> 5
- net col5: track 334.1 -> 29.4 mm, vias 2 -> 1
- net row7: track 349.3 -> 67.6 mm
- net row0: track 378.9 -> 101.7 mm
- net row3: track 420.5 -> 152.3 mm, vias 8 -> 6
- net row1: track 382.7 -> 150.7 mm, vias 7 -> 6
- net col4: track 244.6 -> 34.5 mm, vias 2 -> 1
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Other:
- board size 330.4 x 635.7 mm -> 330.4 x 235.3 mm
- board text added: "ChocoflyMX v1.0 by vitvlkv https://github.com/vlkv/chocofly"
- board text removed: "Chocofly v3.0 by vitvlkv https://github.com/vlkv/chocofly"

Commit message: labels
Parts:
- renumbered SW32 to SW1, SW32 to SW11, SW32 to SW12, SW32 to SW13, SW32 to SW14, SW32 to SW15, SW32 to SW16, SW32 to SW17, SW32 to SW18, SW32 to SW19, SW32 to SW2, SW32 to SW20, SW32 to SW21, SW32 to SW22, SW32 to SW23, SW32 to SW24, SW32 to SW25, SW32 to SW26, SW32 to SW27, SW32 to SW28, SW32 to SW29, SW32 to SW3, SW32 to SW30, SW32 to SW31, SW32 to SW33, SW32 to SW34, SW32 to SW35, SW32 to SW36, SW32 to SW37, SW32 to SW38, SW32 to SW39, SW32 to SW4, SW32 to SW40, SW32 to SW41, SW32 to SW42, SW32 to SW43, SW32 to SW44, SW32 to SW45, SW32 to SW46, SW32 to SW47, SW32 to SW48, SW32 to SW49, SW32 to SW5, SW32 to SW50, SW32 to SW51, SW32 to SW52, SW32 to SW53, SW32 to SW54, SW32 to SW55, SW32 to SW56, SW32 to SW57, SW32 to SW58, SW32 to SW59, SW32 to SW6, SW32 to SW60, SW32 to SW61, SW32 to SW7, SW32 to SW8, SW32 to SW9
Other:
- board text added: "Chocofly v4.0-mx by vitvlkv https://github.com/vlkv/chocofly"
- board text removed: "ChocoflyMX v1.0 by vitvlkv https://github.com/vlkv/chocofly"

Commit message: wip
Connections:
- SW1 pad 1: (no net) -> Net-(D1-A)
- SW1 pad 2: (no net) -> col0
- SW11 pad 1: (no net) -> Net-(D11-A)
- SW11 pad 2: (no net) -> col5
- SW12 pad 1: (no net) -> Net-(D12-A)
- SW12 pad 2: (no net) -> col6
- SW13 pad 1: (no net) -> Net-(D13-A)
- SW13 pad 2: (no net) -> col7
- SW14 pad 1: (no net) -> Net-(D14-A)
- SW14 pad 2: (no net) -> col0
- SW15 pad 1: (no net) -> Net-(D15-A)
- SW15 pad 2: (no net) -> col1
- SW16 pad 1: (no net) -> Net-(D16-A)
- SW16 pad 2: (no net) -> col2
- SW17 pad 1: (no net) -> Net-(D17-A)
- SW17 pad 2: (no net) -> col3
- SW18 pad 1: (no net) -> Net-(D18-A)
- SW18 pad 2: (no net) -> col4
- SW19 pad 1: (no net) -> Net-(D19-A)
- SW19 pad 2: (no net) -> col5
- SW2 pad 1: (no net) -> Net-(D2-A)
- SW2 pad 2: (no net) -> col1
- SW20 pad 1: (no net) -> Net-(D20-A)
- SW20 pad 2: (no net) -> col6
- SW21 pad 1: (no net) -> Net-(D21-A)
- SW21 pad 2: (no net) -> col7
- SW22 pad 1: (no net) -> Net-(D22-A)
- SW22 pad 2: (no net) -> col0
- SW23 pad 1: (no net) -> Net-(D23-A)
- SW23 pad 2: (no net) -> col1
- SW24 pad 1: (no net) -> Net-(D24-A)
- SW24 pad 2: (no net) -> col2
- SW25 pad 1: (no net) -> Net-(D25-A)
- SW25 pad 2: (no net) -> col3
- SW26 pad 1: (no net) -> Net-(D26-A)
- SW26 pad 2: (no net) -> col4
- SW27 pad 1: (no net) -> Net-(D27-A)
- SW27 pad 2: (no net) -> col5
- SW28 pad 1: (no net) -> Net-(D28-A)
- SW28 pad 2: (no net) -> col6
- SW29 pad 1: (no net) -> Net-(D29-A)
- SW29 pad 2: (no net) -> col7
- SW3 pad 1: (no net) -> Net-(D3-A)
- SW3 pad 2: (no net) -> col2
- SW30 pad 1: (no net) -> Net-(D30-A)
- SW30 pad 2: (no net) -> col0
- SW31 pad 1: (no net) -> Net-(D31-A)
- SW31 pad 2: (no net) -> col1
- SW32 pad 1: (no net) -> Net-(D32-A)
- SW32 pad 2: (no net) -> col2
- SW33 pad 1: (no net) -> Net-(D33-A)
- SW33 pad 2: (no net) -> col3
- SW34 pad 1: (no net) -> Net-(D34-A)
- SW34 pad 2: (no net) -> col4
- SW35 pad 1: (no net) -> Net-(D35-A)
- SW35 pad 2: (no net) -> col5
- SW36 pad 1: (no net) -> Net-(D36-A)
- SW36 pad 2: (no net) -> col6
- SW37 pad 1: (no net) -> Net-(D37-A)
- SW37 pad 2: (no net) -> col7
- SW38 pad 1: (no net) -> Net-(D38-A)
- SW38 pad 2: (no net) -> col0
- SW39 pad 1: (no net) -> Net-(D39-A)
- SW39 pad 2: (no net) -> col1
- SW4 pad 1: (no net) -> Net-(D4-A)
- SW4 pad 2: (no net) -> col5
- SW40 pad 1: (no net) -> Net-(D40-A)
- SW40 pad 2: (no net) -> col2
- SW41 pad 1: (no net) -> Net-(D41-A)
- SW41 pad 2: (no net) -> col3
- SW42 pad 1: (no net) -> Net-(D42-A)
- SW42 pad 2: (no net) -> col4
- SW43 pad 1: (no net) -> Net-(D43-A)
- SW43 pad 2: (no net) -> col5
- SW44 pad 1: (no net) -> Net-(D44-A)
- SW44 pad 2: (no net) -> col6
- SW45 pad 1: (no net) -> Net-(D45-A)
- SW45 pad 2: (no net) -> col7
- SW46 pad 1: (no net) -> Net-(D46-A)
- SW46 pad 2: (no net) -> col0
- SW47 pad 1: (no net) -> Net-(D47-A)
- SW47 pad 2: (no net) -> col1
- SW48 pad 1: (no net) -> Net-(D48-A)
- SW48 pad 2: (no net) -> col2
- SW49 pad 1: (no net) -> Net-(D49-A)
- SW49 pad 2: (no net) -> col3
- SW5 pad 1: (no net) -> Net-(D5-A)
- SW5 pad 2: (no net) -> col6
- SW50 pad 1: (no net) -> Net-(D50-A)
- SW50 pad 2: (no net) -> col4
- SW51 pad 1: (no net) -> Net-(D51-A)
- SW51 pad 2: (no net) -> col5
- SW52 pad 1: (no net) -> Net-(D52-A)
- SW52 pad 2: (no net) -> col6
- SW53 pad 1: (no net) -> Net-(D53-A)
- SW53 pad 2: (no net) -> col7
- SW54 pad 1: (no net) -> Net-(D54-A)
- SW54 pad 2: (no net) -> col0
- SW55 pad 1: (no net) -> Net-(D55-A)
- SW55 pad 2: (no net) -> col1
- SW56 pad 1: (no net) -> Net-(D56-A)
- SW56 pad 2: (no net) -> col2
- SW57 pad 1: (no net) -> Net-(D57-A)
- SW57 pad 2: (no net) -> col3
- SW58 pad 1: (no net) -> Net-(D58-A)
- SW58 pad 2: (no net) -> col4
- SW59 pad 1: (no net) -> Net-(D59-A)
- SW59 pad 2: (no net) -> col5
- SW6 pad 1: (no net) -> Net-(D6-A)
- SW6 pad 2: (no net) -> col7
- SW60 pad 1: (no net) -> Net-(D60-A)
- SW60 pad 2: (no net) -> col6
- SW61 pad 1: (no net) -> Net-(D61-A)
- SW61 pad 2: (no net) -> col7
- SW7 pad 1: (no net) -> Net-(D7-A)
- SW7 pad 2: (no net) -> col0
- SW8 pad 1: (no net) -> Net-(D8-A)
- SW8 pad 2: (no net) -> col1
- SW9 pad 1: (no net) -> Net-(D9-A)
- SW9 pad 2: (no net) -> col2
Other:
- board size 330.4 x 235.3 mm -> 330.4 x 146.1 mm
- board text added: "Chocofly v5.0-mx by vitvlkv https://github.com/vlkv/chocofly"
- board text removed: "Chocofly v4.0-mx by vitvlkv https://github.com/vlkv/chocofly"

Commit message: wip
Parts:
- removed SW64: Power, footprints:Switch_MSK-12C01-07
- SW11, SW12, SW13, SW18, SW19, SW20, SW21, SW26, SW27, SW28, SW29, SW34, SW35, SW36, SW37, SW4, SW42, SW43, SW44, SW45, SW5, SW50, SW51, SW52, SW53, SW58, SW59, SW6, SW60, SW61: moved to F.Cu
- moved SW62 18.1 mm to (-20.9, 402.3)
- moved SW63 2.23 mm to (21.3, 400.9)
- moved D6 1.45 mm to (151.1, 387.7)
- turned SW11 to 13.5 degrees
- turned SW12 to 13.5 degrees
- turned SW13 to 9.5 degrees
- turned SW18 to 54 degrees
- turned SW19 to 13.5 degrees
- turned SW20 to 13.5 degrees
- turned SW21 to 9.5 degrees
- turned SW26 to 40.5 degrees
- turned SW27 to 13.5 degrees
- turned SW28 to 13.5 degrees
- turned SW29 to 9.5 degrees
- turned SW34 to 54 degrees
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
Commit message: wip
Parts:
- moved D12 2.50 mm to (89.3, 393.8)
- moved D8 2.50 mm to (-70.8, 398.2)
