File: pcb_mx/chocofly.kicad_pcb (KiCad board)
At the start: 2 copper layers, 330.4 x 146.1 mm, 133 parts, among them P1 battery+, P2 battery-, SW1 SW_Push, SW11 SW_Push, SW12 SW_Push, SW13 SW_Push, SW14 SW_Push, SW15 SW_Push, SW16 SW_Push, SW17 SW_Push, SW18 SW_Push, SW19 SW_Push, SW2 SW_Push, SW20 SW_Push, SW21 SW_Push, SW22 SW_Push, SW23 SW_Push, SW24 SW_Push, SW25 SW_Push, SW26 SW_Push, SW27 SW_Push, SW28 SW_Push, SW29 SW_Push, SW3 SW_Push, SW30 SW_Push, SW31 SW_Push, SW32 SW_Push, SW33 SW_Push, SW34 SW_Push, SW35 SW_Push, SW36 SW_Push, SW37 SW_Push, SW38 SW_Push, SW39 SW_Push, SW4 SW_Push, SW40 SW_Push, SW41 SW_Push, SW42 SW_Push, SW43 SW_Push, SW44 SW_Push, SW45 SW_Push, SW46 SW_Push, SW47 SW_Push, SW48 SW_Push, SW49 SW_Push, SW5 SW_Push, SW50 SW_Push, SW51 SW_Push, SW52 SW_Push, SW53 SW_Push, SW54 SW_Push, SW55 SW_Push, SW56 SW_Push, SW57 SW_Push, SW58 SW_Push, SW59 SW_Push, SW6 SW_Push, SW60 SW_Push, SW61 SW_Push, SW62 Reset, SW63 Power, SW7 SW_Push, SW8 SW_Push, SW9 SW_Push

Commit message: wip on chocomx
Parts:
- removed D10, D62: 1N4148, footprints:diode_TH_SMD
- removed ENC1, ENC2: EVQWGD001_for_mx, footprints:EVQWGD001_for_mx
- removed JP1, JP2: Jumper_NC_Small, footprints:avalanche_Jumper_NC
- removed JP3, JP4: Jumper_NC_Small, footprints:avalanche_Jumper
Connections:
- MCU1 pad 1: encA -> unconnected-(MCU1-TX(PD3)-Pad1)
- MCU1 pad 2: encB -> unconnected-(MCU1-RX(PD2)-Pad2)
Routing:
- net col0: track 22.7 -> 399.7 mm, vias 0 -> 10
- net col1: track 25.0 -> 292.2 mm, vias 0 -> 10
- net col2: track 34.7 -> 278.2 mm, vias 1 -> 9
- net col3: track 36.3 -> 253.4 mm, vias 1 -> 8
- net row4: track 102.0 -> 290.4 mm, vias 5 -> 7
- net row5: track 91.8 -> 263.3 mm, vias 5 -> 6
- net row6: track 77.7 -> 241.5 mm, vias 2 -> 3
- net row2: track 153.3 -> 314.0 mm, vias 5 -> 10
- net row3: track 152.3 -> 304.6 mm, vias 6 -> 11
- net row7: track 67.6 -> 203.1 mm
- net row0: track 101.7 -> 233.1 mm, vias 5 -> 7
- net row1: track 150.7 -> 249.4 mm
- net unconnected-(MCU1-RX(PD2)-Pad2): track 0.00 -> 78.4 mm, vias 0 -> 1
- net encB: track 78.4 -> 0.00 mm, vias 1 -> 0
- net unconnected-(MCU1-TX(PD3)-Pad1): track 0.00 -> 65.2 mm
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
Commit message: wip
Routing:
- net col7: track 27.7 -> 367.4 mm, vias 1 -> 10
- net col6: track 28.6 -> 326.1 mm, vias 1 -> 12
- net col5: track 31.0 -> 287.2 mm, vias 1 -> 10
- net col4: track 34.5 -> 241.5 mm, vias 1 -> 8
- net row4: track 290.4 -> 474.8 mm, vias 7 -> 8
- net row6: track 241.5 -> 418.2 mm, vias 3 -> 6
- net row0: track 233.1 -> 386.5 mm, vias 7 -> 8
- net row7: track 203.1 -> 352.4 mm, vias 1 -> 3
- net row2: track 314.0 -> 460.0 mm, vias 10 -> 13
- net row5: track 263.3 -> 400.8 mm, vias 6 -> 7
- net row3: track 304.6 -> 431.5 mm, vias 11 -> 12
- net row1: track 249.4 -> 350.4 mm, vias 6 -> 8
- net GND: track 130.3 -> 92.5 mm, vias 4 -> 2
- net col2: track 278.2 -> 243.5 mm, vias 9 -> 8
- net Net-(D36-A): track 0.00 -> 27.8 mm
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
Commit message: added encoder back
Parts:
- added D10: 1N4148, footprints:diode_TH_SMD, F.Cu at (-18.4, 470.4)
- added ENC1: EVQWGD001, footprints:EVQWGD001, F.Cu at (-27.9, 464.6)
Connections:
- MCU1 pad 1: unconnected-(MCU1-TX(PD3)-Pad1) -> encA
- MCU1 pad 2: unconnected-(MCU1-RX(PD2)-Pad2) -> encB
Routing:
- net encA: track 0.00 -> 115.6 mm, vias 0 -> 2
- net encB: track 0.00 -> 113.7 mm, vias 0 -> 2
- net unconnected-(MCU1-RX(PD2)-Pad2): track 78.4 -> 0.00 mm, vias 1 -> 0
- net unconnected-(MCU1-TX(PD3)-Pad1): track 65.2 -> 0.00 mm
- net col3: track 253.3 -> 280.3 mm, vias 8 -> 9
- net Net-(D10-A): track 0.00 -> 23.5 mm
- net GND: track 92.5 -> 110.8 mm
- net row1: track 350.4 -> 365.1 mm, vias 8 -> 10
- net row3: track 431.5 -> 439.3 mm, vias 12 -> 13
- net row5: track 400.8 -> 399.1 mm
- net row2: track 460.0 -> 459.4 mm

Commit message: wip
Parts:
- turned ENC1 to 139.5 degrees
Routing:
- net encA: track 115.6 -> 98.3 mm
- net encB: track 113.7 -> 98.5 mm
- net Net-(D10-A): track 23.5 -> 9.93 mm
- net col3: track 280.3 -> 286.6 mm
- net GND: track 110.8 -> 112.9 mm

Commit message: mounting holes added
Parts:
- added H1: MountingHole, MountingHole:MountingHole_2.2mm_M2, F.Cu at (-134.0, 401.2)
- added H10: MountingHole, MountingHole:MountingHole_2.2mm_M2, F.Cu at (64.2, 452.3)
- added H11: MountingHole, MountingHole:MountingHole_2.2mm_M2, F.Cu at (91.8, 404.2)
- added H12: MountingHole, MountingHole:MountingHole_2.2mm_M2, F.Cu at (100.7, 441.2)
- added H13: MountingHole, MountingHole:MountingHole_2.2mm_M2, F.Cu at (134.0, 401.2)
- added H14: MountingHole, MountingHole:MountingHole_2.2mm_M2, F.Cu at (140.3, 438.8)
- added H15: MountingHole, MountingHole:MountingHole_2.2mm_M2, F.Cu at (37.7, 494.1)
- added H16: MountingHole, MountingHole:MountingHole_2.2mm_M2, F.Cu at (76.4, 468.2)
- added H2: MountingHole, MountingHole:MountingHole_2.2mm_M2, F.Cu at (-91.8, 404.2)
- added H3: MountingHole, MountingHole:MountingHole_2.2mm_M2, F.Cu at (-55.3, 415.2)
- added H4: MountingHole, MountingHole:MountingHole_2.2mm_M2, F.Cu at (-140.3, 438.8)
- added H5: MountingHole, MountingHole:MountingHole_2.2mm_M2, F.Cu at (-100.7, 441.2)
- added H6: MountingHole, MountingHole:MountingHole_2.2mm_M2, F.Cu at (-64.2, 452.3)
- added H7: MountingHole, MountingHole:MountingHole_2.2mm_M2, F.Cu at (-37.7, 494.1)
- added H8: MountingHole, MountingHole:MountingHole_2.2mm_M2, F.Cu at (-76.4, 468.2)
- added H9: MountingHole, MountingHole:MountingHole_2.2mm_M2, F.Cu at (55.3, 415.2)
- moved D28 5.78 mm to (94.5, 415.5)
- moved D60 5.78 mm to (103.4, 452.5)
- moved D48 5.28 mm to (-66.8, 463.4)
- moved D16 5.28 mm to (-57.9, 426.3)
- moved D34 4.20 mm to (45.3, 502.4)
- moved D50 4.20 mm to (79.5, 479.1)
- moved D57 4.20 mm to (-81.2, 478.4)
- moved D29 4.20 mm to (135.9, 412.4)
- moved D61 4.20 mm to (142.2, 450.0)
- moved D47 4.20 mm to (-103.6, 453.4)
- moved D46 4.20 mm to (-142.2, 450.0)
- moved D41 4.20 mm to (-46.5, 501.1)
- moved D14 3.59 mm to (-135.8, 411.8)
- moved D59 3.28 mm to (66.8, 463.4)
- moved D27 3.28 mm to (57.9, 426.3)
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Routing:
- net row6: track 418.2 -> 406.0 mm
- net row3: track 439.3 -> 448.7 mm
- net row2: track 459.4 -> 465.9 mm
- net row7: track 352.4 -> 358.6 mm
- net col2: track 243.5 -> 249.6 mm
- net Net-(D9-A): track 21.6 -> 27.2 mm
- net Net-(D56-A): track 21.6 -> 27.2 mm
- net Net-(D24-A): track 22.0 -> 27.6 mm
- net Net-(D40-A): track 21.7 -> 27.3 mm
- net col5: track 287.2 -> 292.8 mm
- net row4: track 474.7 -> 480.1 mm
- net col7: track 367.4 -> 369.9 mm
- net Net-(D14-A): track 27.7 -> 25.3 mm
- net col1: track 292.2 -> 294.3 mm
- net Net-(D47-A): track 28.4 -> 26.3 mm
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
Commit message: pcb is generally done
Routing:
- net col5: track 292.8 -> 314.1 mm
- net row6: track 406.0 -> 410.7 mm
- net col2: track 249.6 -> 250.7 mm
- net row0: track 386.5 -> 385.6 mm
