File: chocofly_mx_pcb/chocofly.kicad_pcb (KiCad board)
At the start: 2 copper layers, 330.4 x 146.1 mm, 143 parts, among them P1 battery+, P2 battery-, SW1 SW_Push, SW11 SW_Push, SW12 SW_Push, SW13 SW_Push, SW14 SW_Push, SW15 SW_Push, SW16 SW_Push, SW17 SW_Push, SW18 SW_Push, SW19 SW_Push, SW2 SW_Push, SW20 SW_Push, SW21 SW_Push, SW22 SW_Push, SW23 SW_Push, SW24 SW_Push, SW25 SW_Push, SW26 SW_Push, SW27 SW_Push, SW28 SW_Push, SW29 SW_Push, SW3 SW_Push, SW30 SW_Push, SW31 SW_Push, SW32 SW_Push, SW33 SW_Push, SW34 SW_Push, SW35 SW_Push, SW36 SW_Push, SW37 SW_Push, SW38 SW_Push, SW39 SW_Push, SW4 SW_Push, SW40 SW_Push, SW41 SW_Push, SW42 SW_Push, SW43 SW_Push, SW44 SW_Push, SW45 SW_Push, SW46 SW_Push, SW47 SW_Push, SW48 SW_Push, SW49 SW_Push, SW5 SW_Push, SW50 SW_Push, SW51 SW_Push, SW52 SW_Push, SW53 SW_Push, SW54 SW_Push, SW55 SW_Push, SW56 SW_Push, SW57 SW_Push, SW58 SW_Push, SW59 SW_Push, SW6 SW_Push, SW60 SW_Push, SW61 SW_Push, SW62 Reset, SW63 Power, SW7 SW_Push, SW8 SW_Push, SW9 SW_Push

Commit message: wip
Routing:
- net GND: vias 2 -> 48
- added copper zone on B.Cu, net GND
- added copper zone on F.Cu, net GND

Commit message: using non-hotswap footprint
Parts:
- SW1, SW11, SW12, SW13, SW14, SW15, SW16, SW17, SW18, SW19, SW2, SW20, SW21, SW22, SW23, SW24, SW25, SW26, SW27, SW28, SW29, SW3, SW30, SW31, SW32, SW33, SW34, SW35, SW36, SW37, SW38, SW39, SW4, SW40, SW41, SW42, SW43, SW44, SW45, SW46, SW47, SW48, SW49, SW5, SW50, SW51, SW52, SW53, SW54, SW55, SW56, SW57, SW58, SW59, SW6, SW60, SW61, SW7, SW8, SW9: footprint footprints:CherryMX_MidHeight_Hotswap_1u -> footprints:MyCherryMX_1u
Routing:
- net col5: track 314.1 -> 191.4 mm, vias 10 -> 7
- net col2: track 250.7 -> 132.4 mm, vias 8 -> 4
- net col6: track 326.7 -> 212.0 mm, vias 12 -> 9
- net col7: track 369.6 -> 256.1 mm, vias 10 -> 7
- net col0: track 401.3 -> 289.2 mm, vias 10 -> 6
- net col1: track 294.3 -> 183.5 mm, vias 10 -> 6
- net col4: track 241.3 -> 154.7 mm, vias 8 -> 7
- net col3: track 286.4 -> 202.4 mm, vias 9 -> 7
- net Net-(D16-A): track 26.9 -> 2.54 mm
- net Net-(D46-A): track 26.9 -> 2.65 mm
- net Net-(D41-A): track 27.9 -> 3.61 mm
- net Net-(D48-A): track 27.0 -> 2.94 mm
- net Net-(D28-A): track 26.5 -> 2.72 mm
- net Net-(D47-A): track 26.3 -> 2.65 mm
- net Net-(D60-A): track 26.3 -> 2.72 mm
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Other:
- board text added: "ChocoflyMX v5.0 by vitvlkv https://github.com/vlkv/chocofly"
- board text removed: "Chocofly v5.0-mx by vitvlkv https://github.com/vlkv/chocofly"
