File: chocofly_glp_pcb/chocofly.kicad_pcb (KiCad board)
At the start: 2 copper layers, 330.4 x 146.1 mm, 143 parts, among them P1 battery+, P2 battery-, SW1 SW_Push, SW11 SW_Push, SW12 SW_Push, SW13 SW_Push, SW14 SW_Push, SW15 SW_Push, SW16 SW_Push, SW17 SW_Push, SW18 SW_Push, SW19 SW_Push, SW2 SW_Push, SW20 SW_Push, SW21 SW_Push, SW22 SW_Push, SW23 SW_Push, SW24 SW_Push, SW25 SW_Push, SW26 SW_Push, SW27 SW_Push, SW28 SW_Push, SW29 SW_Push, SW3 SW_Push, SW30 SW_Push, SW31 SW_Push, SW32 SW_Push, SW33 SW_Push, SW34 SW_Push, SW35 SW_Push, SW36 SW_Push, SW37 SW_Push, SW38 SW_Push, SW39 SW_Push, SW4 SW_Push, SW40 SW_Push, SW41 SW_Push, SW42 SW_Push, SW43 SW_Push, SW44 SW_Push, SW45 SW_Push, SW46 SW_Push, SW47 SW_Push, SW48 SW_Push, SW49 SW_Push, SW5 SW_Push, SW50 SW_Push, SW51 SW_Push, SW52 SW_Push, SW53 SW_Push, SW54 SW_Push, SW55 SW_Push, SW56 SW_Push, SW57 SW_Push, SW58 SW_Push, SW59 SW_Push, SW6 SW_Push, SW60 SW_Push, SW61 SW_Push, SW62 Reset, SW63 Power, SW7 SW_Push, SW8 SW_Push, SW9 SW_Push

Commit message: wip
Parts:
- moved D44 0.80 mm to (97.8, 429.2)
- moved D27 0.78 mm to (57.8, 425.5)
- moved D59 0.60 mm to (66.7, 462.8)
Routing:
- net col7: track 18.8 -> 336.5 mm, vias 7 -> 2
- net col5: track 73.2 -> 256.2 mm, vias 5 -> 2
- net col6: track 118.4 -> 300.0 mm, vias 9 -> 4
- net col4: track 94.5 -> 271.0 mm, vias 7 -> 2
- net col3: track 101.4 -> 222.7 mm, vias 4 -> 2
- net row1: track 265.6 -> 376.3 mm
- net row7: track 255.1 -> 360.1 mm
- net row5: track 302.3 -> 405.9 mm, vias 6 -> 9
- net row3: track 359.9 -> 451.6 mm
- net row4: track 437.5 -> 478.8 mm
- net Net-(D34-A): track 0.00 -> 26.1 mm
- net Net-(D60-A): track 0.00 -> 26.0 mm
- net Net-(D28-A): track 0.00 -> 26.0 mm
- net Net-(D59-A): track 0.00 -> 25.3 mm
- net Net-(D27-A): track 0.00 -> 25.3 mm
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
Commit message: wip
Parts:
- moved D47 0.32 mm to (-103.1, 451.3)
- moved D15 0.29 mm to (-94.3, 414.3)
- moved D14 0.21 mm to (-135.8, 412.0)
Routing:
- net col0: track 200.1 -> 297.7 mm
- net col1: track 184.2 -> 249.5 mm, vias 2 -> 0
- net col2: track 151.2 -> 203.2 mm
- net row2: track 428.0 -> 471.1 mm
- net Net-(D25-A): track 11.8 -> 25.0 mm
- net row6: track 410.1 -> 415.8 mm
- net col6: track 300.0 -> 301.8 mm
- net Net-(D14-A): track 25.1 -> 25.7 mm
- net col7: track 336.5 -> 337.1 mm
- net row5: track 405.9 -> 405.6 mm, vias 9 -> 10

Commit message: done
Routing:
- net col4: track 270.8 -> 267.8 mm
- net row2: track 471.1 -> 473.9 mm
- net row1: track 376.3 -> 378.3 mm
- net col1: track 249.5 -> 251.2 mm
- net row0: track 386.2 -> 387.4 mm
- net row3: track 451.8 -> 453.0 mm
- net col2: track 203.2 -> 204.3 mm
- net GND: vias 3 -> 2
Other:
- outline, holes or cut-outs redrawn

Commit message: wip
Routing:
- net GND: vias 2 -> 70
