File: chocofly_mx_top_plate/chocofly.kicad_pcb (KiCad board)
At the start: 2 copper layers, 330.4 x 146.1 mm, 77 parts, among them SW1 SW_Push, SW10 SW_Push, SW11 SW_Push, SW12 SW_Push, SW13 SW_Push, SW14 SW_Push, SW15 SW_Push, SW16 SW_Push, SW17 SW_Push, SW18 SW_Push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

Commit message: wip
Other:
- board text added: "ATTENTION: Need 1.2 mm plate thikness otherwise switches won't click in."
